Commit message: fixed the urdf

File: urdf/relay.urdf.xacro (robot description, xacro)
@@ -83,5 +83,5 @@
     <parent link="base_link"/>
     <child link="top_link"/>
-    <origin xyz="0 0 0"/>
+    <origin xyz="0 0 0.18906"/>
 </joint>
 <link name="rwheel_link">
@@ -103,4 +103,14 @@
       <gravity value="True"/>
       <!-- <material>Gazebo/Red</material> -->
+      <surface>
+        <friction>
+          <ode>
+            <mu>1</mu>
+            <mu2>1</mu2>
+            <slip1>0</slip1>
+            <slip2>0</slip2>
+          </ode>
+        </friction>
+      </surface>
 </gazebo>
 <joint name="scooter_right_wheel_joint" type="continuous">
@@ -110,5 +120,5 @@
     <parent link="base_link"/>
     <child link="rwheel_link"/>
-    <origin xyz="0 0 0"/>
+    <origin xyz="0 0.16189 0"/>
 </joint>
  <transmission name="scooter_right_wheel_trans">
@@ -140,4 +150,14 @@
       <gravity value="True"/>
       <!-- <material>Gazebo/Red</material> -->
+      <surface>
+        <friction>
+          <ode>
+            <mu>1</mu>
+            <mu2>1</mu2>
+            <slip1>0</slip1>
+            <slip2>0</slip2>
+          </ode>
+        </friction>
+      </surface>
 </gazebo>
 <joint name="scooter_left_wheel_joint" type="continuous">
@@ -147,5 +167,5 @@
     <parent link="base_link"/>
     <child link="lwheel_link"/>
-    <origin xyz="0 0 0"/>
+    <origin xyz="0 -0.16189 0"/>
 </joint>
  <transmission name="scooter_left_wheel_trans">
@@ -177,4 +197,14 @@
       <gravity value="True"/>
       <!-- <material>Gazebo/Red</material> -->
+      <surface>
+        <friction>
+          <ode>
+            <mu>0</mu>
+            <mu2>0</mu2>
+            <slip1>1</slip1>
+            <slip2>1</slip2>
+          </ode>
+        </friction>
+      </surface>
 </gazebo>
 <joint name="caster_front_wheel_joint" type="fixed">
@@ -184,5 +214,5 @@
     <parent link="base_link"/>
     <child link="fcaster_link"/>
-    <origin xyz="0 0 0"/>
+    <origin xyz="0.16189 0 0.0008"/>
 </joint>
 <link name="bcaster_link">
@@ -204,4 +234,14 @@
       <gravity value="True"/>
       <!-- <material>Gazebo/Red</material> -->
+      <surface>
+        <friction>
+          <ode>
+            <mu>0</mu>
+            <mu2>0</mu2>
+            <slip1>1</slip1>
+            <slip2>1</slip2>
+          </ode>
+        </friction>
+      </surface>
 </gazebo>
 <joint name="caster_back_wheel_joint" type="fixed">
@@ -211,5 +251,5 @@
     <parent link="base_link"/>
     <child link="bcaster_link"/>
-    <origin xyz="0 0 0"/>
+    <origin xyz="-0.16189 0 0.0008"/>
 </joint>
 <gazebo>

Commit message: changed params

File: urdf/relay.urdf.xacro (robot description, xacro)
@@ -117,5 +117,5 @@
     <axis xyz="0 1 0" rpy="0 0 0" />
     <dynamics damping="0.20" friction="0.0"/>
-    <limit effort="10000" velocity="30"/>
+    <limit effort="100" velocity="10"/>
     <parent link="base_link"/>
     <child link="rwheel_link"/>
@@ -164,5 +164,5 @@
     <axis xyz="0 1 0" rpy="0 0 0" />
     <dynamics damping="0.20" friction="0.0"/>
-    <limit effort="10000" velocity="30"/>
+    <limit effort="100" velocity="10"/>
     <parent link="base_link"/>
     <child link="lwheel_link"/>

Commit message: fixed the params as per urdf

File: urdf/relay.urdf.xacro (robot description, xacro)
@@ -1,4 +1,4 @@
 <?xml version="1.0"?>
-<robot name="relay" xmlns:xacro="http://ros.org/wiki/xacro">
+<robot name="intel_robot" xmlns:xacro="http://ros.org/wiki/xacro">
 <xacro:property name="bodyrad" value="0.1"/>
 <xacro:property name="baselen" value="0.1"/>
@@ -116,9 +116,11 @@
 <joint name="scooter_right_wheel_joint" type="continuous">
     <axis xyz="0 1 0" rpy="0 0 0" />
-    <dynamics damping="0.20" friction="0.0"/>
-    <limit effort="100" velocity="10"/>
+    <dynamics damping="0.10" friction="0.0"/>
+    <!-- since we have wheel radius = 0.05 meters and max linear speed 2.5 m/s
+     thus max angular velocity of  wheel is w = v/r = 50  -->
+    <limit effort="100000000" velocity="50"/>
     <parent link="base_link"/>
     <child link="rwheel_link"/>
-    <origin xyz="0 0.16189 0"/>
+    <origin xyz="0 -0.16189 0"/>
 </joint>
  <transmission name="scooter_right_wheel_trans">
@@ -163,9 +165,11 @@
 <joint name="scooter_left_wheel_joint" type="continuous">
     <axis xyz="0 1 0" rpy="0 0 0" />
-    <dynamics damping="0.20" friction="0.0"/>
-    <limit effort="100" velocity="10"/>
+    <dynamics damping="0.10" friction="0.0"/>
+    <!-- since we have wheel radius = 0.05 meters and max linear speed 2.5 m/s
+     thus max angular velocity of  wheel is w = v/r = 50  -->
+    <limit effort="100000000" velocity="50"/>
     <parent link="base_link"/>
     <child link="lwheel_link"/>
-    <origin xyz="0 -0.16189 0"/>
+    <origin xyz="0 0.16189 0"/>
 </joint>
  <transmission name="scooter_left_wheel_trans">
@@ -256,4 +260,5 @@
     <plugin name="gazebo_ros_control" filename="libgazebo_ros_control.so">
       <robotNamespace>/</robotNamespace>
+      <robotSimType>gazebo_ros_control/DefaultRobotHWSim</robotSimType>
     </plugin>
   </gazebo>

Commit message: changed paras

File: urdf/relay.urdf.xacro (robot description, xacro)
@@ -98,5 +98,5 @@
       </geometry>
    </collision>
-   <xacro:cylinder_inertia m ="0.1" r="0.05" h="0.05" />
+   <xacro:cylinder_inertia m ="0.08" r="0.05" h="0.05" />
 </link>
 <gazebo reference="rwheel_link">
@@ -116,8 +116,8 @@
 <joint name="scooter_right_wheel_joint" type="continuous">
     <axis xyz="0 1 0" rpy="0 0 0" />
-    <dynamics damping="0.10" friction="0.0"/>
+    <dynamics damping="0.0" friction="0.0"/>
     <!-- since we have wheel radius = 0.05 meters and max linear speed 2.5 m/s
      thus max angular velocity of  wheel is w = v/r = 50  -->
-    <limit effort="100000000" velocity="50"/>
+    <limit effort="10" velocity="50"/>
     <parent link="base_link"/>
     <child link="rwheel_link"/>
@@ -147,5 +147,5 @@
       </geometry>
    </collision>
-   <xacro:cylinder_inertia m ="0.1" r="0.05" h="0.05" />
+   <xacro:cylinder_inertia m ="0.08" r="0.05" h="0.05" />
 </link>
 <gazebo reference="lwheel_link">
@@ -165,8 +165,8 @@
 <joint name="scooter_left_wheel_joint" type="continuous">
     <axis xyz="0 1 0" rpy="0 0 0" />
-    <dynamics damping="0.10" friction="0.0"/>
+    <dynamics damping="0.0" friction="0.0"/>
     <!-- since we have wheel radius = 0.05 meters and max linear speed 2.5 m/s
      thus max angular velocity of  wheel is w = v/r = 50  -->
-    <limit effort="100000000" velocity="50"/>
+    <limit effort="10" velocity="50"/>
     <parent link="base_link"/>
     <child link="lwheel_link"/>
@@ -196,5 +196,5 @@
       </geometry>
    </collision>
-   <xacro:sphere_inertia m ="0.1" r="0.05" />
+   <xacro:sphere_inertia m ="0.08" r="0.05" />
 </link>
 <gazebo reference="fcaster_link">
@@ -204,8 +204,8 @@
         <friction>
           <ode>
-            <mu>0</mu>
-            <mu2>0</mu2>
-            <slip1>1</slip1>
-            <slip2>1</slip2>
+            <mu>0.0</mu>
+            <mu2>0.0</mu2>
+            <slip1>1.0</slip1>
+            <slip2>1.0</slip2>
           </ode>
         </friction>
@@ -214,6 +214,5 @@
 <joint name="caster_front_wheel_joint" type="fixed">
     <!-- <axis xyz="0 0 0" rpy="0 0 0" /> -->
-    <dynamics damping="0.20" friction="0.0"/>
-    <limit effort="10000" velocity="30"/>
+    <dynamics damping="0.0" friction="0.0"/>
     <parent link="base_link"/>
     <child link="fcaster_link"/>
@@ -233,5 +232,5 @@
       </geometry>
    </collision>
-   <xacro:sphere_inertia m ="0.1" r="0.05" />
+   <xacro:sphere_inertia m ="0.08" r="0.05" />
 </link>
 <gazebo reference="bcaster_link">
@@ -241,8 +240,8 @@
         <friction>
           <ode>
-            <mu>0</mu>
-            <mu2>0</mu2>
-            <slip1>1</slip1>
-            <slip2>1</slip2>
+            <mu>0.0</mu>
+            <mu2>0.0</mu2>
+            <slip1>1.0</slip1>
+            <slip2>1.0</slip2>
           </ode>
         </friction>
@@ -251,6 +250,5 @@
 <joint name="caster_back_wheel_joint" type="fixed">
     <!-- <axis xyz="0 0 0" rpy="0 0 0" /> -->
-    <dynamics damping="0.20" friction="0.0"/>
-    <limit effort="10000" velocity="30"/>
+    <dynamics damping="0.0" friction="0.0"/>
     <parent link="base_link"/>
     <child link="bcaster_link"/>
