Commit message: Added experimental bare bone straight line cruise control

File: urdf/intel_robot.urdf.xacro (robot description, xacro)
@@ -1,7 +1,7 @@
 <?xml version="1.0"?>
-<robot name="roscontrol" xmlns:xacro="http://ros.org/wiki/xacro">
+<robot name="intel_robot" xmlns:xacro="http://ros.org/wiki/xacro">
 <xacro:property name="bodyrad" value="0.1"/>
 <xacro:property name="baselen" value="0.1"/>
-<xacro:property name="base_mass" value="1"/>
+<xacro:property name="base_mass" value="2"/>
 <xacro:property name="toplen" value="0.5"/>
 <xacro:property name="top_mass" value="8"/>
@@ -9,6 +9,5 @@
 <xacro:property name="wheelwidth" value="0.025"/>
 <xacro:property name="casterrad" value="0.012"/>
-<xacro:property name="caster_mass" value="0.2"/>
-<xacro:property name="pi" value="3.1415"/>
+<xacro:property name="caster_mass" value="0.01"/>
 <xacro:property name="wheel_mass" value="0.2"/>
  <xacro:macro name="default_inertial" params="mass">
@@ -35,22 +34,12 @@
 </xacro:macro>
 <xacro:macro name="caster" params="suffix reflect">
-<!--link name="${suffix}_caster"-->
+<link name="${suffix}_caster_link">
   <visual>
    <geometry>
      <sphere radius="${casterrad}"/>
      </geometry>
-     <origin rpy="0 0 0" xyz="${reflect*0.0875} 0 -0.062"/>
+     <origin rpy="0 0 0" xyz="${reflect*0.0875} 0 -0.0625"/>
      <material name="black"/>
     </visual>
-    <surface>
-            <friction>
-              <ode>
-                <mu>0</mu>
-                <mu2>0</mu2>
-                <slip1>1.0</slip1>
-                <slip2>1.0</slip2>
-              </ode>
-            </friction>
-          </surface>
     <collision>
     <origin rpy="0  0  0" xyz="${reflect*0.0875} 0 -0.0625"/>
@@ -59,29 +48,7 @@
       </geometry>
     </collision>
-   <xacro:sphere_inertia m="${caster_mass}" r="${casterrad}"/>
-  <!--/link-->
- <!--joint name="${suffix}_caster_to_wheel" type="fixed">
-    <parent link="base_link"/>
-    <child link="${suffix}_caster"/>
-    <origin xyz="${reflect*0.0875} 0 -0.06"/>
-    <dynamics damping="0.0" friction="0.0" implicitSpringDamper="True"/>
-  </joint-->
-<!--gazebo reference="${suffix}_caster">
-      <mu1 value="200.0"/>
-      <mu2 value="100.0"/>
-      <kp value="10000000.0" />
-      <kd value="1.0" />
-      <material>Gazebo/Grey</material>
-    </gazebo-->
-  <!--transmission name="${suffix}_caster_trans">
-    <type>transmission_interface/SimpleTransmission</type>
-    <actuator name="${suffix}_caster_motor">
-      <mechanicalReduction>1</mechanicalReduction>
-    </actuator>
-    <joint name="${suffix}_caster_joint">
-    <hardwareInterface>VelocityJointInterface</hardwareInterface>
-    </joint>
-  </transmission-->
-</xacro:macro>
+  <xacro:sphere_inertia m="${caster_mass}" r="${casterrad}"/>
+</link>
+ </xacro:macro>
 <link name="base_link">
     <visual>
@@ -97,12 +64,95 @@
       </geometry>
     </collision>
-<xacro:cylinder_inertia m="${top_mass}" r="${bodyrad}" h="${baselen}"/>
-  <xacro:caster suffix="front" reflect="1"/>
-  <xacro:caster suffix="back" reflect="-1"/>
+  <!--xacro:caster suffix="front" reflect="1"/>
+  <xacro:caster suffix="back" reflect="-1"/-->
   </link>
- <gazebo reference="base_link">
-      <gravity value="True"/>
-      <material>Gazebo/Blue</material>
-    </gazebo>
+  <gazebo reference="base_link">
+    <gravity>true</gravity>
+    <material>Gazebo/Blue</material>
+    <sensor name="imu_sensor" type="imu">
+      <always_on>true</always_on>
+      <update_rate>100</update_rate>
+      <visualize>true</visualize>
+      <topic>__default_topic__</topic>
+      <plugin filename="libgazebo_ros_imu_sensor.so" name="imu_plugin">
+        <topicName>imu</topicName>
+        <bodyName>imu_link</bodyName>
+        <updateRateHZ>10.0</updateRateHZ>
+        <gaussianNoise>0.0</gaussianNoise>
+        <xyzOffset>0 0 0</xyzOffset>
+        <rpyOffset>0 0 0</rpyOffset>
+        <frameName>imu_link</frameName>
+      </plugin>
+      <pose>0 0 0 0 0 0</pose>
+    </sensor>
+  </gazebo>
+<xacro:caster suffix="front" reflect="1"/>
+<joint name="casterf_to_base" type="fixed">
+    <axis xyz="1 1 1"/>
+    <parent link="base_link"/>
+    <child link="front_caster_link"/>
+    <origin xyz="0 0 0"/>
+</joint>
+<xacro:caster suffix="back" reflect="-1"/>
+<gazebo reference="front_caster_link">
+      <surface>
+            <friction>
+              <ode>
+                <mu>0.11</mu>
+                <mu2>0.11</mu2>
+                <slip1>0.5</slip1>
+                <slip2>0.5</slip2>
+              </ode>
+            </friction>
+          </surface>
+      <!--mu1 value="0.0"/>
+      <mu2 value="0.0"/>
+      <kp value="10000000.0" />
+      <kd value="1.0" /-->
+      <material>Gazebo/Black</material>
+     </gazebo>
+    <!--transmission name="front_caster_wheel_trans">
+       <type>transmission_interface/SimpleTransmission</type>
+       <actuator name="front_caster_wheel_motor">
+         <hardwareInterface>EffortJointInterface</hardwareInterface>
+         <mechanicalReduction>1</mechanicalReduction>
+       </actuator>
+       <joint name="casterf_to_base">
+          <hardwareInterface>VelocityJointInterface</hardwareInterface>
+       </joint>
+  </transmission-->
+<joint name="casterb_to_base" type="fixed">
+    <axis xyz="1 1 1"/>
+    <parent link="base_link"/>
+    <child link="back_caster_link"/>
+    <origin xyz="0 0 0"/>
+</joint>
+<gazebo reference="back_caster_link">
+     <surface>
+            <friction>
+              <ode>
+                <mu>0.11</mu>
+                <mu2>0.11</mu2>
+                <slip1>0.5</slip1>
+                <slip2>0.5</slip2>
+              </ode>
+            </friction>
+          </surface>
+      <!--mu1 value="0.0"/>
+      <mu2 value="0.0"/>
+      <kp value="10000000.0" />
+      <kd value="1.0" /-->
+      <material>Gazebo/Black</material>
+     </gazebo>
+    <!--transmission name="back_caster_wheel_trans">
+       <type>transmission_interface/SimpleTransmission</type>
+       <actuator name="back_caster_wheel_motor">
+         <hardwareInterface>EffortJointInterface</hardwareInterface>
+         <mechanicalReduction>1</mechanicalReduction>
+       </actuator>
+       <joint name="casterb_to_base">
+          <hardwareInterface>VelocityJointInterface</hardwareInterface>
+       </joint>
+  </transmission-->
 <link name="top_link">
     <visual>
@@ -155,19 +205,19 @@
     </joint>
     <gazebo reference="${prefix}_${suffix}_wheel">
-      <mu1 value="200.0"/>
-      <mu2 value="100.0"/>
+      <mu1 value="1.0"/>
+      <mu2 value="1.0"/>
       <kp value="10000000.0" />
       <kd value="1.0" />
       <material>Gazebo/Black</material>
-    </gazebo>
-  <transmission name="${prefix}_${suffix}_wheel_trans">
-    <type>transmission_interface/SimpleTransmission</type>
-    <actuator name="${prefix}_${suffix}_wheel_motor">
-    <hardwareInterface>EffortJointInterface</hardwareInterface>
-      <mechanicalReduction>1</mechanicalReduction>
-    </actuator>
-    <joint name="${prefix}_${suffix}_wheel_joint">
-    <hardwareInterface>VelocityJointInterface</hardwareInterface>
-    </joint>
+     </gazebo>
+    <transmission name="${prefix}_${suffix}_wheel_trans">
+       <type>transmission_interface/SimpleTransmission</type>
+       <actuator name="${prefix}_${suffix}_wheel_motor">
+         <hardwareInterface>EffortJointInterface</hardwareInterface>
+         <mechanicalReduction>1</mechanicalReduction>
+       </actuator>
+       <joint name="${prefix}_${suffix}_wheel_joint">
+          <hardwareInterface>hardware_interface/VelocityJointInterface</hardwareInterface>
+       </joint>
   </transmission>
  </xacro:macro>

Commit message: update 1

File: urdf/intel_robot.urdf.xacro (robot description, xacro)
@@ -1,7 +1,7 @@
 <?xml version="1.0"?>
-<robot name="intel_robot" xmlns:xacro="http://ros.org/wiki/xacro">
+<robot name="roscontrol" xmlns:xacro="http://ros.org/wiki/xacro">
 <xacro:property name="bodyrad" value="0.1"/>
 <xacro:property name="baselen" value="0.1"/>
-<xacro:property name="base_mass" value="2"/>
+<xacro:property name="base_mass" value="1"/>
 <xacro:property name="toplen" value="0.5"/>
 <xacro:property name="top_mass" value="8"/>
@@ -9,5 +9,6 @@
 <xacro:property name="wheelwidth" value="0.025"/>
 <xacro:property name="casterrad" value="0.012"/>
-<xacro:property name="caster_mass" value="0.01"/>
+<xacro:property name="caster_mass" value="0.2"/>
+<xacro:property name="pi" value="3.1415"/>
 <xacro:property name="wheel_mass" value="0.2"/>
  <xacro:macro name="default_inertial" params="mass">
@@ -34,21 +35,53 @@
 </xacro:macro>
 <xacro:macro name="caster" params="suffix reflect">
-<link name="${suffix}_caster_link">
+<!--link name="${suffix}_caster"-->
   <visual>
    <geometry>
      <sphere radius="${casterrad}"/>
      </geometry>
-     <origin rpy="0 0 0" xyz="${reflect*0.0875} 0 -0.0625"/>
+     <origin rpy="0 0 0" xyz="${reflect*0.0875} 0 -0.0626"/>
      <material name="black"/>
     </visual>
+    <surface>
+            <friction>
+              <ode>
+                <mu>0</mu>
+                <mu2>0</mu2>
+                <slip1>1.0</slip1>
+                <slip2>1.0</slip2>
+              </ode>
+            </friction>
+          </surface>
     <collision>
-    <origin rpy="0  0  0" xyz="${reflect*0.0875} 0 -0.0625"/>
+    <origin rpy="0  0  0" xyz="${reflect*0.0875} 0 -0.0626"/>
       <geometry>
         <sphere radius="${casterrad}" />
       </geometry>
     </collision>
-  <xacro:sphere_inertia m="${caster_mass}" r="${casterrad}"/>
-</link>
- </xacro:macro>
+   <xacro:sphere_inertia m="${caster_mass}" r="${casterrad}"/>
+  <!--/link-->
+ <!--joint name="${suffix}_caster_to_wheel" type="fixed">
+    <parent link="base_link"/>
+    <child link="${suffix}_caster"/>
+    <origin xyz="${reflect*0.0875} 0 -0.06"/>
+    <dynamics damping="0.0" friction="0.0" implicitSpringDamper="True"/>
+  </joint-->
+<!--gazebo reference="${suffix}_caster">
+      <mu1 value="200.0"/>
+      <mu2 value="100.0"/>
+      <kp value="10000000.0" />
+      <kd value="1.0" />
+      <material>Gazebo/Grey</material>
+    </gazebo-->
+  <!--transmission name="${suffix}_caster_trans">
+    <type>transmission_interface/SimpleTransmission</type>
+    <actuator name="${suffix}_caster_motor">
+      <mechanicalReduction>1</mechanicalReduction>
+    </actuator>
+    <joint name="${suffix}_caster_joint">
+    <hardwareInterface>VelocityJointInterface</hardwareInterface>
+    </joint>
+  </transmission-->
+</xacro:macro>
 <link name="base_link">
     <visual>
@@ -99,8 +132,8 @@
             <friction>
               <ode>
-                <mu>0.11</mu>
-                <mu2>0.11</mu2>
-                <slip1>0.5</slip1>
-                <slip2>0.5</slip2>
+                <mu>0.005</mu>
+                <mu2>0.005</mu2>
+                <!-- <slip1>1</slip1>
+                <slip2>1</slip2> -->
               </ode>
             </friction>
@@ -132,8 +165,8 @@
             <friction>
               <ode>
-                <mu>0.11</mu>
-                <mu2>0.11</mu2>
-                <slip1>0.5</slip1>
-                <slip2>0.5</slip2>
+                <mu>1</mu>
+                <mu2>1</mu2>
+                <!-- <slip1>0.5</slip1>
+                <slip2>0.5</slip2> -->
               </ode>
             </friction>
@@ -155,4 +188,11 @@
        </joint>
   </transmission-->
+  <xacro:caster suffix="front" reflect="1"/>
+  <xacro:caster suffix="back" reflect="-1"/>
+  </link>
+ <gazebo reference="base_link">
+      <gravity value="True"/>
+      <material>Gazebo/Blue</material>
+    </gazebo>
 <link name="top_link">
     <visual>
@@ -201,23 +241,23 @@
       <child link="${prefix}_${suffix}_wheel"/>
       <origin xyz="0 ${reflect*0.1126} -0.05" rpy="0 0 0"/>
-       <dynamics damping="0.20" friction="0.90"/>
-      <limit effort="1000000" velocity="1000000"/>
+       <dynamics damping="0.20" friction="0.0"/>
+      <limit effort="1000000" velocity="1"/>
     </joint>
     <gazebo reference="${prefix}_${suffix}_wheel">
-      <mu1 value="1.0"/>
-      <mu2 value="1.0"/>
+      <mu1 value="200.0"/>
+      <mu2 value="100.0"/>
       <kp value="10000000.0" />
       <kd value="1.0" />
       <material>Gazebo/Black</material>
-     </gazebo>
-    <transmission name="${prefix}_${suffix}_wheel_trans">
-       <type>transmission_interface/SimpleTransmission</type>
-       <actuator name="${prefix}_${suffix}_wheel_motor">
-         <hardwareInterface>EffortJointInterface</hardwareInterface>
-         <mechanicalReduction>1</mechanicalReduction>
-       </actuator>
-       <joint name="${prefix}_${suffix}_wheel_joint">
-          <hardwareInterface>hardware_interface/VelocityJointInterface</hardwareInterface>
-       </joint>
+    </gazebo>
+  <transmission name="${prefix}_${suffix}_wheel_trans">
+    <type>transmission_interface/SimpleTransmission</type>
+    <actuator name="${prefix}_${suffix}_wheel_motor">
+    <hardwareInterface>EffortJointInterface</hardwareInterface>
+      <mechanicalReduction>1</mechanicalReduction>
+    </actuator>
+    <joint name="${prefix}_${suffix}_wheel_joint">
+    <hardwareInterface>VelocityJointInterface</hardwareInterface>
+    </joint>
   </transmission>
  </xacro:macro>

Commit message: added propoer link parameter for caster wheel

File: urdf/intel_robot.urdf.xacro (robot description, xacro)
@@ -10,5 +10,4 @@
 <xacro:property name="casterrad" value="0.012"/>
 <xacro:property name="caster_mass" value="0.2"/>
-<xacro:property name="pi" value="3.1415"/>
 <xacro:property name="wheel_mass" value="0.2"/>
  <xacro:macro name="default_inertial" params="mass">
@@ -35,5 +34,5 @@
 </xacro:macro>
 <xacro:macro name="caster" params="suffix reflect">
-<!--link name="${suffix}_caster"-->
+<link name="${suffix}_caster_link">
   <visual>
    <geometry>
@@ -60,27 +59,5 @@
     </collision>
    <xacro:sphere_inertia m="${caster_mass}" r="${casterrad}"/>
-  <!--/link-->
- <!--joint name="${suffix}_caster_to_wheel" type="fixed">
-    <parent link="base_link"/>
-    <child link="${suffix}_caster"/>
-    <origin xyz="${reflect*0.0875} 0 -0.06"/>
-    <dynamics damping="0.0" friction="0.0" implicitSpringDamper="True"/>
-  </joint-->
-<!--gazebo reference="${suffix}_caster">
-      <mu1 value="200.0"/>
-      <mu2 value="100.0"/>
-      <kp value="10000000.0" />
-      <kd value="1.0" />
-      <material>Gazebo/Grey</material>
-    </gazebo-->
-  <!--transmission name="${suffix}_caster_trans">
-    <type>transmission_interface/SimpleTransmission</type>
-    <actuator name="${suffix}_caster_motor">
-      <mechanicalReduction>1</mechanicalReduction>
-    </actuator>
-    <joint name="${suffix}_caster_joint">
-    <hardwareInterface>VelocityJointInterface</hardwareInterface>
-    </joint>
-  </transmission-->
+  </link>
 </xacro:macro>
 <link name="base_link">
@@ -97,6 +74,4 @@
       </geometry>
     </collision>
-  <!--xacro:caster suffix="front" reflect="1"/>
-  <xacro:caster suffix="back" reflect="-1"/-->
   </link>
   <gazebo reference="base_link">
@@ -127,5 +102,4 @@
     <origin xyz="0 0 0"/>
 </joint>
-<xacro:caster suffix="back" reflect="-1"/>
 <gazebo reference="front_caster_link">
       <surface>
@@ -139,20 +113,7 @@
             </friction>
           </surface>
-      <!--mu1 value="0.0"/>
-      <mu2 value="0.0"/>
-      <kp value="10000000.0" />
-      <kd value="1.0" /-->
       <material>Gazebo/Black</material>
      </gazebo>
-    <!--transmission name="front_caster_wheel_trans">
-       <type>transmission_interface/SimpleTransmission</type>
-       <actuator name="front_caster_wheel_motor">
-         <hardwareInterface>EffortJointInterface</hardwareInterface>
-         <mechanicalReduction>1</mechanicalReduction>
-       </actuator>
-       <joint name="casterf_to_base">
-          <hardwareInterface>VelocityJointInterface</hardwareInterface>
-       </joint>
-  </transmission-->
+<xacro:caster suffix="back" reflect="-1"/>
 <joint name="casterb_to_base" type="fixed">
     <axis xyz="1 1 1"/>
@@ -165,6 +126,6 @@
             <friction>
               <ode>
-                <mu>1</mu>
-                <mu2>1</mu2>
+                <mu>0.005</mu>
+                <mu2>0.005</mu2>
                 <!-- <slip1>0.5</slip1>
                 <slip2>0.5</slip2> -->
@@ -172,27 +133,6 @@
             </friction>
           </surface>
-      <!--mu1 value="0.0"/>
-      <mu2 value="0.0"/>
-      <kp value="10000000.0" />
-      <kd value="1.0" /-->
       <material>Gazebo/Black</material>
      </gazebo>
-    <!--transmission name="back_caster_wheel_trans">
-       <type>transmission_interface/SimpleTransmission</type>
-       <actuator name="back_caster_wheel_motor">
-         <hardwareInterface>EffortJointInterface</hardwareInterface>
-         <mechanicalReduction>1</mechanicalReduction>
-       </actuator>
-       <joint name="casterb_to_base">
-          <hardwareInterface>VelocityJointInterface</hardwareInterface>
-       </joint>
-  </transmission-->
-  <xacro:caster suffix="front" reflect="1"/>
-  <xacro:caster suffix="back" reflect="-1"/>
-  </link>
- <gazebo reference="base_link">
-      <gravity value="True"/>
-      <material>Gazebo/Blue</material>
-    </gazebo>
 <link name="top_link">
     <visual>
@@ -258,5 +198,5 @@
     </actuator>
     <joint name="${prefix}_${suffix}_wheel_joint">
-    <hardwareInterface>VelocityJointInterface</hardwareInterface>
+    <hardwareInterface>hardware_interface/VelocityJointInterface</hardwareInterface>
     </joint>
   </transmission>

Commit message: changed friction and velcocity of joints

File: urdf/intel_robot.urdf.xacro (robot description, xacro)
@@ -182,5 +182,5 @@
       <origin xyz="0 ${reflect*0.1126} -0.05" rpy="0 0 0"/>
        <dynamics damping="0.20" friction="0.0"/>
-      <limit effort="1000000" velocity="1"/>
+      <limit effort="100" velocity="20"/>
     </joint>
     <gazebo reference="${prefix}_${suffix}_wheel">

Commit message: big fix

File: urdf/intel_robot.urdf.xacro (robot description, xacro)
@@ -39,5 +39,5 @@
      <sphere radius="${casterrad}"/>
      </geometry>
-     <origin rpy="0 0 0" xyz="${reflect*0.0875} 0 -0.0626"/>
+     <origin rpy="0 0 0" xyz="${reflect*0.0875} 0 -0.0624"/>
      <material name="black"/>
     </visual>
@@ -45,13 +45,13 @@
             <friction>
               <ode>
-                <mu>0</mu>
-                <mu2>0</mu2>
-                <slip1>1.0</slip1>
-                <slip2>1.0</slip2>
+                <mu>0.0</mu>
+                <mu2>0.0</mu2>
+                <!-- <slip1>1.0</slip1>
+                <slip2>1.0</slip2> -->
               </ode>
             </friction>
           </surface>
     <collision>
-    <origin rpy="0  0  0" xyz="${reflect*0.0875} 0 -0.0626"/>
+    <origin rpy="0  0  0" xyz="${reflect*0.0875} 0 -0.0624"/>
       <geometry>
         <sphere radius="${casterrad}" />
@@ -181,6 +181,6 @@
       <child link="${prefix}_${suffix}_wheel"/>
       <origin xyz="0 ${reflect*0.1126} -0.05" rpy="0 0 0"/>
-       <dynamics damping="0.20" friction="0.0"/>
-      <limit effort="100" velocity="20"/>
+      <dynamics damping="0.20" friction="0.0"/>
+      <limit effort="10000" velocity="30"/>
     </joint>
     <gazebo reference="${prefix}_${suffix}_wheel">
